File: breakout.kicad_pcb (KiCad board)
At the start: 2 copper layers, 65 x 30 mm, 24 parts, among them J1 GPIO, J2 Conn_01x01, J3 Conn_01x01, J4 Conn_01x01, J6 BO, J8 Conn_01x04_Female, J9 Conn_01x04_Female, P1 Conn_01x01, P2 Conn_01x01, P3 Conn_01x01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

Commit message: add url
Other:
- board text added: "github.com/asssaf/pwm-breakout-phat v1.0"
Changed lines of the file:
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@@
     (property "ki_keywords" "connector")
     (attr through_hole)
-    (fp_text reference "J1" (at 2.5 0 180) (layer "B.SilkS")
+    (fp_text reference "J1" (at 0.516927 2.619663 180) (layer "B.SilkS")
         (effects (font (size 1 1) (thickness 0.15)) (justify mirror))
     )
@@
     (effects (font (size 1 1) (thickness 0.15)) (justify left bottom mirror))
   )
+  (gr_text "github.com/asssaf/pwm-breakout-phat  v1.0" (at 158.71279 78.405575) (layer "B.SilkS")
+    (effects (font (size 1.5 1.5) (thickness 0.3) bold) (justify left bottom mirror))
+  )
   (gr_text "5V" (at 102.265096 85.562625) (layer "B.SilkS")
