File: breakout.kicad_pcb (KiCad board)
At the start: 2 copper layers, 65 x 30 mm, 24 parts, among them J1 GPIO, J2 Conn_01x01, J3 Conn_01x01, J4 Conn_01x01, J6 BO, J8 Conn_01x04_Female, J9 Conn_01x04_Female, P1 Conn_01x01, P2 Conn_01x01, P3 Conn_01x01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

Commit message: cleanup
Parts:
- removed U3: ATtiny85-20S, Package_SO:SOIC-8W_5.3x5.3mm_P1.27mm
Changed lines of the file:
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@@
   (net 39 "unconnected-(P8-Pin_1-Pad1)")
   (net 40 "unconnected-(P9-Pin_1-Pad1)")
-  (net 41 "unconnected-(U3-~{RESET}{slash}PB5-Pad1)")
-  (net 42 "unconnected-(U3-XTAL1{slash}PB3-Pad2)")
-  (net 43 "unconnected-(U3-XTAL2{slash}PB4-Pad3)")
-  (net 44 "unconnected-(U3-GND-Pad4)")
-  (net 45 "unconnected-(U3-AREF{slash}PB0-Pad5)")
-  (net 46 "unconnected-(U3-PB1-Pad6)")
-  (net 47 "unconnected-(U3-PB2-Pad7)")
-  (net 48 "unconnected-(U3-VCC-Pad8)")
-  (net 49 "/I2CVCC")
+  (net 41 "/I2CVCC")
   (footprint "Mine2:ConnectedPads_01x04" (layer "F.Cu")
     (at 129.880337 93.066927 90)
@@
       (net 1 "GND") (pinfunction "Pin_1") (pintype "passive"))
     (pad "2" smd roundrect (at -0.5 1.325) (size 0.6 1.55) (layers "F.Cu" "F.Paste" "F.Mask") (roundrect_rratio 0.25)
-      (net 49 "/I2CVCC") (pinfunction "Pin_2") (pintype "passive"))
+      (net 41 "/I2CVCC") (pinfunction "Pin_2") (pintype "passive"))
     (pad "3" smd roundrect (at 0.5 1.325) (size 0.6 1.55) (layers "F.Cu" "F.Paste" "F.Mask") (roundrect_rratio 0.25)
       (net 2 "/GPIO[2]{slash}SDA1") (pinfunction "Pin_3") (pintype "passive"))
@@
       (net 1 "GND") (pinfunction "Pin_1") (pintype "passive"))
     (pad "2" smd roundrect (at -0.5 1.325) (size 0.6 1.55) (layers "F.Cu" "F.Paste" "F.Mask") (roundrect_rratio 0.25)
-      (net 49 "/I2CVCC") (pinfunction "Pin_2") (pintype "passive"))
+      (net 41 "/I2CVCC") (pinfunction "Pin_2") (pintype "passive"))
     (pad "3" smd roundrect (at 0.5 1.325) (size 0.6 1.55) (layers "F.Cu" "F.Paste" "F.Mask") (roundrect_rratio 0.25)
       (net 2 "/GPIO[2]{slash}SDA1") (pinfunction "Pin_3") (pintype "passive"))
@@
       (stroke (width 0.05) (type solid)) (fill none) (layer "F.CrtYd"))
     (pad "" np_thru_hole circle locked (at 0 0) (size 2.7 2.7) (drill 2.7) (layers "*.Cu" "*.Mask"))
-  )
-  (footprint "Package_SO:SOIC-8W_5.3x5.3mm_P1.27mm" (layer "F.Cu")
-    (at 4.775 2.975)
-    (descr "8-Lead Plastic Small Outline (SM) - 5.28 mm Body [SOIC] (http://ww1.microchip.com/downloads/en/PackagingSpec/00000049BQ.pdf)")
-    (tags "SOIC 1.27")
-    (property "Sheetfile" "breakout.kicad_sch")
-    (property "Sheetname" "")
-    (property "ki_description" "20MHz, 8kB Flash, 512B SRAM, 512B EEPROM, debugWIRE, SOIC-8W")
-    (property "ki_keywords" "AVR 8bit Microcontroller tinyAVR")
-    (attr smd)
-    (fp_text reference "U3" (at 0 -3.68) (layer "F.SilkS")
-        (effects (font (size 1 1) (thickness 0.15)))
-    )
-    (fp_text value "ATtiny85-20S" (at 0 3.68) (layer "F.Fab")
-        (effects (font (size 1 1) (thickness 0.15)))
-    )
-    (fp_text user "${REFERENCE}" (at 0 0) (layer "F.Fab")
-        (effects (font (size 1 1) (thickness 0.15)))
-    )
-    (fp_line (start -2.75 -2.755) (end -2.75 -2.55)
-      (stroke (width 0.15) (type solid)) (layer "F.SilkS"))
-    (fp_line (start -2.75 -2.755) (end 2.75 -2.755)
-      (stroke (width 0.15) (type solid)) (layer "F.SilkS"))
-    (fp_line (start -2.75 -2.55) (end -4.5 -2.55)
-      (stroke (width 0.15) (type solid)) (layer "F.SilkS"))
-    (fp_line (start -2.75 2.755) (end -2.75 2.455)
-      (stroke (width 0.15) (type solid)) (layer "F.SilkS"))
-    (fp_line (start -2.75 2.755) (end 2.75 2.755)
-      (stroke (width 0.15) (type solid)) (layer "F.SilkS"))
-    (fp_line (start 2.75 -2.755) (end 2.75 -2.455)
-      (stroke (width 0.15) (type solid)) (layer "F.SilkS"))
-    (fp_line (start 2.75 2.755) (end 2.75 2.455)
-      (stroke (width 0.15) (type solid)) (layer "F.SilkS"))
-    (fp_line (start -4.75 -2.95) (end -4.75 2.95)
-      (stroke (width 0.05) (type solid)) (layer "F.CrtYd"))
-    (fp_line (start -4.75 -2.95) (end 4.75 -2.95)
-      (stroke (width 0.05) (type solid)) (layer "F.CrtYd"))
-    (fp_line (start -4.75 2.95) (end 4.75 2.95)
-      (stroke (width 0.05) (type solid)) (layer "F.CrtYd"))
-    (fp_line (start 4.75 -2.95) (end 4.75 2.95)
-      (stroke (width 0.05) (type solid)) (layer "F.CrtYd"))
-    (fp_line (start -2.65 -1.65) (end -1.65 -2.65)
-      (stroke (width 0.15) (type solid)) (layer "F.Fab"))
-    (fp_line (start -2.65 2.65) (end -2.65 -1.65)
-      (stroke (width 0.15) (type solid)) (layer "F.Fab"))
-    (fp_line (start -1.65 -2.65) (end 2.65 -2.65)
-      (stroke (width 0.15) (type solid)) (layer "F.Fab"))
-    (fp_line (start 2.65 -2.65) (end 2.65 2.65)
-      (stroke (width 0.15) (type solid)) (layer "F.Fab"))
-    (fp_line (start 2.65 2.65) (end -2.65 2.65)
-      (stroke (width 0.15) (type solid)) (layer "F.Fab"))
-    (pad "1" smd rect (at -3.65 -1.905) (size 1.7 0.65) (layers "F.Cu" "F.Paste" "F.Mask")
-      (net 41 "unconnected-(U3-~{RESET}{slash}PB5-Pad1)") (pinfunction "~{RESET}/PB5") (pintype "bidirectional"))
-    (pad "2" smd rect (at -3.65 -0.635) (size 1.7 0.65) (layers "F.Cu" "F.Paste" "F.Mask")
-      (net 42 "unconnected-(U3-XTAL1{slash}PB3-Pad2)") (pinfunction "XTAL1/PB3") (pintype "bidirectional"))
-    (pad "3" smd rect (at -3.65 0.635) (size 1.7 0.65) (layers "F.Cu" "F.Paste" "F.Mask")
-      (net 43 "unconnected-(U3-XTAL2{slash}PB4-Pad3)") (pinfunction "XTAL2/PB4") (pintype "bidirectional"))
-    (pad "4" smd rect (at -3.65 1.905) (size 1.7 0.65) (layers "F.Cu" "F.Paste" "F.Mask")
-      (net 44 "unconnected-(U3-GND-Pad4)") (pinfunction "GND") (pintype "power_in"))
-    (pad "5" smd rect (at 3.65 1.905) (size 1.7 0.65) (layers "F.Cu" "F.Paste" "F.Mask")
-      (net 45 "unconnected-(U3-AREF{slash}PB0-Pad5)") (pinfunction "AREF/PB0") (pintype "bidirectional"))
-    (pad "6" smd rect (at 3.65 0.635) (size 1.7 0.65) (layers "F.Cu" "F.Paste" "F.Mask")
-      (net 46 "unconnected-(U3-PB1-Pad6)") (pinfunction "PB1") (pintype "bidirectional"))
-    (pad "7" smd rect (at 3.65 -0.635) (size 1.7 0.65) (layers "F.Cu" "F.Paste" "F.Mask")
-      (net 47 "unconnected-(U3-PB2-Pad7)") (pinfunction "PB2") (pintype "bidirectional"))
-    (pad "8" smd rect (at 3.65 -1.905) (size 1.7 0.65) (layers "F.Cu" "F.Paste" "F.Mask")
-      (net 48 "unconnected-(U3-VCC-Pad8)") (pinfunction "VCC") (pintype "power_in"))
-    (model "${KICAD6_3DMODEL_DIR}/Package_SO.3dshapes/SOIC-8W_5.3x5.3mm_P1.27mm.wrl"
-      (offset (xyz 0 0 0))
-      (scale (xyz 1 1 1))
-      (rotate (xyz 0 0 0))
-    )
   )
   (footprint "MountingHole:MountingHole_2.7mm_M2.5" locked (layer "F.Cu")
@@
       ))
     (pad "2" smd rect (at 0 0 180) (size 1 1.5) (layers "B.Cu" "B.Mask")
-      (net 49 "/I2CVCC") (pinfunction "C") (pintype "passive"))
+      (net 41 "/I2CVCC") (pinfunction "C") (pintype "passive"))
     (pad "3" smd custom (at 1.3 0 180) (size 1 0.5) (layers "B.Cu" "B.Mask")
       (net 30 "+5V") (pinfunction "B") (pintype "passive") (zone_connect 2)
@@
   (segment (start 129.845 90.475) (end 129.845 93.015) (width 0.2) (layer "B.Cu") (net 40))
   (segment (start 129.845 85.395) (end 129.845 87.935) (width 0.2) (layer "B.Cu") (net 40))
-  (segment (start 102.930133 82.400088) (end 102.930133 83.16206) (width 0.5) (layer "F.Cu") (net 49))
-  (segment (start 103.944747 86.720253) (end 103.945 86.72) (width 0.2) (layer "F.Cu") (net 49))
-  (segment (start 103.945 84.176927) (end 103.945 86.72) (width 0.5) (layer "F.Cu") (net 49))
-  (segment (start 103.944747 92.124046) (end 103.944747 86.720253) (width 0.5) (layer "F.Cu") (net 49))
-  (segment (start 102.930133 83.16206) (end 103.945 84.176927) (width 0.5) (layer "F.Cu") (net 49))
-  (via (at 102.930133 82.400088) (size 0.9) (drill 0.6) (layers "F.Cu" "B.Cu") (net 49))
-  (segment (start 104.391925 84.99344) (end 104.391925 83.86188) (width 0.5) (layer "B.Cu") (net 49))
-  (segment (start 104.391925 83.86188) (end 102.930133 82.400088) (width 0.5) (layer "B.Cu") (net 49))
+  (segment (start 102.930133 82.400088) (end 102.930133 83.16206) (width 0.5) (layer "F.Cu") (net 41))
+  (segment (start 103.944747 86.720253) (end 103.945 86.72) (width 0.2) (layer "F.Cu") (net 41))
+  (segment (start 103.945 84.176927) (end 103.945 86.72) (width 0.5) (layer "F.Cu") (net 41))
+  (segment (start 103.944747 92.124046) (end 103.944747 86.720253) (width 0.5) (layer "F.Cu") (net 41))
+  (segment (start 102.930133 83.16206) (end 103.945 84.176927) (width 0.5) (layer "F.Cu") (net 41))
+  (via (at 102.930133 82.400088) (size 0.9) (drill 0.6) (layers "F.Cu" "B.Cu") (net 41))
+  (segment (start 104.391925 84.99344) (end 104.391925 83.86188) (width 0.5) (layer "B.Cu") (net 41))
+  (segment (start 104.391925 83.86188) (end 102.930133 82.400088) (width 0.5) (layer "B.Cu") (net 41))
   (zone locked (net 0) (net_name "") (layers "F&B.Cu") (name "NoFillCircle") (hatch edge 0.5)
     (connect_pads (clearance 0))
