File: breakout.kicad_sch (KiCad schematic)
At the start: 23 parts, among them J1 GPIO, J2 Conn_01x01, J3 Conn_01x01, J4 Conn_01x01, J6 BO, J8 Conn_01x04_Female, J9 Conn_01x04_Female, P1 Conn_01x01, P2 Conn_01x01, P3 Conn_01x01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

Commit message: add LCSC Part Number
Parts:
- J8, J9: LCSC Part Number (none) -> C495539
Changed lines of the file:
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@@
+      (effects (font (size 1.27 1.27)) hide)
+    )
+    (property "LCSC Part Number" "C495539" (at 92.71 110.49 0)
       (effects (font (size 1.27 1.27)) hide)
     )
@@
       (effects (font (size 1.27 1.27)) hide)
     )
+    (property "LCSC Part Number" "C495539" (at 92.71 127 0)
+      (effects (font (size 1.27 1.27)) hide)
+    )
